Commit message: update aim sdk

File: legged_robot_description/g1_description/urdf/g1_29dof_lock_waist_rev_1_0.urdf (robot description, URDF)
Before this commit: robot g1, 39 links, 38 joints
Links:
- added link gripper_tcp; visual sphere radius=0.005
Joints:
- added joint gripper_tcp_joint: type fixed, parent right_wrist_yaw_link, child gripper_tcp, origin xyz=0.173 0.007 0.0 rpy=0 0 0

File: legged_robot_description/g1_description/urdf/g1_29dof_lock_waist_rev_1_0.urdf.xacro (robot description, xacro)
@@ -4,4 +4,5 @@
   <xacro:arg name="network_interface" default="lo" />
   <xacro:arg name="use_sim" default="true" />
+  <xacro:arg name="use_mock_components" default="false" />
   <xacro:include filename="$(find g1_description)/urdf/g1_29dof_lock_waist_rev_1_0_macro.urdf.xacro" />
   <xacro:include filename="$(find g1_description)/urdf/g1_29dof_lock_waist_rev_1_0.ros2_control.xacro" />
@@ -11,3 +12,13 @@
     network_interface="$(arg network_interface)"
     use_sim="$(arg use_sim)"/>
+   <!-- Gipper URDF -->
+  <xacro:include filename="$(find g1_description)/urdf/inspire_gripper_macro.xacro" />
+  <!-- Link gripper with right arm -->
+  <xacro:inspire_gripper name="right" parent_link="right_wrist_yaw_link" use_sim="$(arg use_sim)" use_mock_components="$(arg use_mock_components)" serial_port="/dev/ttyUSB0">
+    <origin xyz="0.02 0 0" rpy="0 1.5708 0" />
+  </xacro:inspire_gripper>
+  <!-- Link gripper with left arm -->
+  <xacro:inspire_gripper name="left" parent_link="left_wrist_yaw_link" use_sim="$(arg use_sim)" use_mock_components="$(arg use_mock_components)" serial_port="/dev/ttyUSB1">
+    <origin xyz="0.02 0 0" rpy="0 1.5708 0" />
+  </xacro:inspire_gripper>
 </robot>

File: legged_robot_description/g1_description/urdf/g1_29dof_lock_waist_rev_1_0_macro.urdf.xacro (robot description, xacro)
@@ -943,4 +943,17 @@
     </collision>
   </link>
+  <!-- gripper_tcp -->
+  <link name="gripper_tcp">
+    <visual>
+      <geometry>
+        <sphere radius="0.005"/>
+      </geometry>
+    </visual>
+  </link>
+  <joint name="gripper_tcp_joint" type="fixed">
+    <parent link="right_wrist_yaw_link"/>
+    <child link="gripper_tcp"/>
+    <origin xyz="0.173 0.007 0.0" rpy="0 0 0"/>
+  </joint>
   </xacro:macro>
 </robot>
