Commit message: various update

File: legged_robot_description/g1_description/urdf/g1_29dof_lock_waist_rev_1_0.ros2_control.xacro (robot description, xacro)
@@ -1,17 +1,10 @@
 <?xml version="1.0"?>
 <robot xmlns:xacro="http://www.ros.org/wiki/xacro">
-  <xacro:macro name="g1_29dof_lock_waist_rev_1_0_ros2_control" params="prefix enable_sim:=false network_interface:=lo">
+  <xacro:macro name="g1_29dof_lock_waist_rev_1_0_ros2_control" params="prefix network_interface:=lo">
     <ros2_control name="g1_29dof_lock_waist_rev_1_0_ros2_control" type="system" is_async="true">
-      <xacro:if value="${enable_sim}">
-        <hardware>
-          <plugin>legged_ros2_control/MujocoSystemInterface</plugin>
-        </hardware>
-      </xacro:if>
-      <xacro:unless value="${enable_sim}">
-        <hardware>
-          <plugin>legged_ros2_control/G1SystemInterface</plugin>
-          <param name="network_interface">${network_interface}</param>
-        </hardware>
-      </xacro:unless>
+      <hardware>
+        <plugin>legged_ros2_control/G1SystemInterface</plugin>
+        <param name="network_interface">${network_interface}</param>
+      </hardware>
       <joint name="${prefix}left_hip_pitch_joint">
         <command_interface name="position">
@@ -527,17 +520,4 @@
         <state_interface name="effort" />
       </joint>
-      <xacro:if value="${enable_sim}">
-        <sensor name="imu-torso">
-          <state_interface name="orientation.x"/>
-          <state_interface name="orientation.y"/>
-          <state_interface name="orientation.z"/>
-          <state_interface name="orientation.w"/>
-          <state_interface name="angular_velocity.x"/>
-          <state_interface name="angular_velocity.y"/>
-          <state_interface name="angular_velocity.z"/>
-          <state_interface name="linear_acceleration.x"/>
-          <state_interface name="linear_acceleration.y"/>
-          <state_interface name="linear_acceleration.z"/>
-        </sensor>
         <sensor name="imu-pelvis">
           <state_interface name="orientation.x"/>
@@ -552,19 +532,4 @@
           <state_interface name="linear_acceleration.z"/>
         </sensor>
-      </xacro:if>
-      <xacro:unless value="${enable_sim}">
-        <sensor name="imu-pelvis">
-          <state_interface name="orientation.x"/>
-          <state_interface name="orientation.y"/>
-          <state_interface name="orientation.z"/>
-          <state_interface name="orientation.w"/>
-          <state_interface name="angular_velocity.x"/>
-          <state_interface name="angular_velocity.y"/>
-          <state_interface name="angular_velocity.z"/>
-          <state_interface name="linear_acceleration.x"/>
-          <state_interface name="linear_acceleration.y"/>
-          <state_interface name="linear_acceleration.z"/>
-        </sensor>
-      </xacro:unless>
     </ros2_control>
   </xacro:macro>

File: legged_robot_description/g1_description/urdf/g1_29dof_lock_waist_rev_1_0.urdf.xacro (robot description, xacro)
@@ -2,5 +2,4 @@
 <robot xmlns:xacro="http://www.ros.org/wiki/xacro" name="g1_29dof_lock_waist_rev_1_0">
   <xacro:arg name="prefix" default="" />
-  <xacro:arg name="enable_sim" default="true" />
   <xacro:arg name="network_interface" default="lo" />
   <xacro:include filename="$(find g1_description)/urdf/g1_29dof_lock_waist_rev_1_0_macro.urdf.xacro" />
@@ -9,5 +8,4 @@
   <xacro:g1_29dof_lock_waist_rev_1_0_ros2_control
     prefix="$(arg prefix)"
-    enable_sim="$(arg enable_sim)"
     network_interface="$(arg network_interface)"/>
 </robot>
