Commit message: various updates

File: legged_robot_description/g1_description/urdf/g1_29dof_lock_waist_rev_1_0.ros2_control.xacro (robot description, xacro)
@@ -1,6 +1,6 @@
 <?xml version="1.0"?>
 <robot xmlns:xacro="http://www.ros.org/wiki/xacro">
-  <xacro:macro name="g1_29dof_lock_waist_rev_1_0_ros2_control" params="prefix network_interface:=lo">
-    <ros2_control name="g1_29dof_lock_waist_rev_1_0_ros2_control" type="system" is_async="true">
+  <xacro:macro name="g1_ros2_control" params="prefix network_interface:=lo">
+    <ros2_control name="g1_ros2_control" type="system" is_async="true">
       <hardware>
         <plugin>legged_ros2_control/G1SystemInterface</plugin>

File: legged_robot_description/g1_description/urdf/g1_29dof_lock_waist_rev_1_0.urdf (robot description, URDF)
Before this commit: robot g1_29dof_lock_waist_rev_1_0, 39 links, 38 joints
Links:
- link head_link: geometry collision mesh filename=package://g1_description/urdf/meshes/head_link.STL; visual mesh filename=package://g1_description/urdf/meshes/head_link.STL
- link left_ankle_pitch_link: geometry collision mesh filename=package://g1_description/urdf/meshes/left_ankle_pitch_link.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; visual mesh filename=package://g1_description/urdf/meshes/left_ankle_pitch_link.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
- link left_ankle_roll_link: geometry collision sphere radius=0.005; collision sphere radius=0.005
- link left_elbow_link: geometry collision mesh filename=package://g1_description/urdf/meshes/left_elbow_link.STL; visual mesh filename=package://g1_description/urdf/meshes/left_elbow_link.STL
- link left_hip_pitch_link: geometry collision mesh filename=package://g1_description/urdf/meshes/left_hip_pitch_link.STL; visual mesh filename=package://g1_description/urdf/meshes/left_hip_pitch_link.STL
- link left_hip_roll_link: geometry collision mesh filename=package://g1_description/urdf/meshes/left_hip_roll_link.STL; visual mesh filename=package://g1_description/urdf/meshes/left_hip_roll_link.STL
- link left_hip_yaw_link: geometry collision mesh filename=package://g1_description/urdf/meshes/left_hip_yaw_link.STL; visual mesh filename=package://g1_description/urdf/meshes/left_hip_yaw_link.STL
- link left_knee_link: geometry collision mesh filename=package://g1_description/urdf/meshes/left_knee_link.STL; visual mesh filename=package://g1_description/urdf/meshes/left_knee_link.STL
- link left_rubber_hand: geometry visual mesh filename=package://g1_description/urdf/meshes/left_rubber_hand.STL
- link left_shoulder_pitch_link: geometry collision cylinder length=0.05 radius=0.03; visual mesh filename=package://g1_description/urdf/meshes/left_shoulder_pitch_li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
- link left_shoulder_roll_link: geometry collision cylinder length=0.03 radius=0.03; visual mesh filename=package://g1_description/urdf/meshes/left_shoulder_roll_lin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
- link left_shoulder_yaw_link: geometry collision mesh filename=package://g1_description/urdf/meshes/left_shoulder_yaw_link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; visual mesh filename=package://g1_description/urdf/meshes/left_shoulder_yaw_link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
- link left_wrist_pitch_link: geometry collision mesh filename=package://g1_description/urdf/meshes/left_wrist_pitch_link.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; visual mesh filename=package://g1_description/urdf/meshes/left_wrist_pitch_link.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
- link left_wrist_roll_link: geometry collision mesh filename=package://g1_description/urdf/meshes/left_wrist_roll_link.S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; visual mesh filename=package://g1_description/urdf/meshes/left_wrist_roll_link.S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
- link left_wrist_yaw_link: geometry collision mesh filename=package://g1_description/urdf/meshes/left_wrist_yaw_link.STL; visual mesh filename=package://g1_description/urdf/meshes/left_wrist_yaw_link.STL
- link logo_link: geometry collision mesh filename=package://g1_description/urdf/meshes/logo_link.STL; visual mesh filename=package://g1_description/urdf/meshes/logo_link.STL
- link pelvis: geometry visual mesh filename=package://g1_description/urdf/meshes/pelvis.STL
- link pelvis_contour_link: geometry collision mesh filename=package://g1_description/urdf/meshes/pelvis_contour_link.STL; visual mesh filename=package://g1_description/urdf/meshes/pelvis_contour_link.STL
- link right_ankle_pitch_link: geometry collision mesh filename=package://g1_description/urdf/meshes/right_ankle_pitch_link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; visual mesh filename=package://g1_description/urdf/meshes/right_ankle_pitch_link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
- link right_ankle_roll_link: geometry collision sphere radius=0.005; collision sphere radius=0.005
- link right_elbow_link: geometry collision mesh filename=package://g1_description/urdf/meshes/right_elbow_link.STL; visual mesh filename=package://g1_description/urdf/meshes/right_elbow_link.STL
- link right_hip_pitch_link: geometry collision mesh filename=package://g1_description/urdf/meshes/right_hip_pitch_link.S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; visual mesh filename=package://g1_description/urdf/meshes/right_hip_pitch_link.S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
- link right_hip_roll_link: geometry collision mesh filename=package://g1_description/urdf/meshes/right_hip_roll_link.STL; visual mesh filename=package://g1_description/urdf/meshes/right_hip_roll_link.STL
- link right_hip_yaw_link: geometry collision mesh filename=package://g1_description/urdf/meshes/right_hip_yaw_link.STL; visual mesh filename=package://g1_description/urdf/meshes/right_hip_yaw_link.STL
- link right_knee_link: geometry collision mesh filename=package://g1_description/urdf/meshes/right_knee_link.STL; visual mesh filename=package://g1_description/urdf/meshes/right_knee_link.STL
- link right_rubber_hand: geometry visual mesh filename=package://g1_description/urdf/meshes/right_rubber_hand.STL
- link right_shoulder_pitch_link: geometry collision cylinder length=0.05 radius=0.03; visual mesh filename=package://g1_description/urdf/meshes/right_shoulder_pitch_l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
- link right_shoulder_roll_link: geometry collision cylinder length=0.03 radius=0.03; visual mesh filename=package://g1_description/urdf/meshes/right_shoulder_roll_li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
- link right_shoulder_yaw_link: geometry collision mesh filename=package://g1_description/urdf/meshes/right_shoulder_yaw_lin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; visual mesh filename=package://g1_description/urdf/meshes/right_shoulder_yaw_lin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
- link right_wrist_pitch_link: geometry collision mesh filename=package://g1_description/urdf/meshes/right_wrist_pitch_link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; visual mesh filename=package://g1_description/urdf/meshes/right_wrist_pitch_link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
- link right_wrist_roll_link: geometry collision mesh filename=package://g1_description/urdf/meshes/right_wrist_roll_link.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; visual mesh filename=package://g1_description/urdf/meshes/right_wrist_roll_link.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
- link right_wrist_yaw_link: geometry collision mesh filename=package://g1_description/urdf/meshes/right_wrist_yaw_link.S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; visual mesh filename=package://g1_description/urdf/meshes/right_wrist_yaw_link.S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
- link torso_link: geometry collision mesh filename=package://g1_description/urdf/meshes/torso_link_rev_1_0.STL; visual mesh filename=package://g1_description/urdf/meshes/torso_link_rev_1_0.STL
- link waist_roll_link: geometry visual mesh filename=package://g1_description/urdf/meshes/waist_roll_link_rev_1_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
- link waist_yaw_link: geometry visual mesh filename=package://g1_description/urdf/meshes/waist_yaw_link_rev_1_0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

File: legged_robot_description/g1_description/urdf/g1_29dof_lock_waist_rev_1_0.urdf.xacro (robot description, xacro)
@@ -1,10 +1,10 @@
 <?xml version="1.0"?>
-<robot xmlns:xacro="http://www.ros.org/wiki/xacro" name="g1_29dof_lock_waist_rev_1_0">
+<robot xmlns:xacro="http://www.ros.org/wiki/xacro" name="g1">
   <xacro:arg name="prefix" default="" />
   <xacro:arg name="network_interface" default="lo" />
   <xacro:include filename="$(find g1_description)/urdf/g1_29dof_lock_waist_rev_1_0_macro.urdf.xacro" />
   <xacro:include filename="$(find g1_description)/urdf/g1_29dof_lock_waist_rev_1_0.ros2_control.xacro" />
-  <xacro:g1_29dof_lock_waist_rev_1_0 prefix="$(arg prefix)" />
-  <xacro:g1_29dof_lock_waist_rev_1_0_ros2_control
+  <xacro:g1 prefix="$(arg prefix)" />
+  <xacro:g1_ros2_control
     prefix="$(arg prefix)"
     network_interface="$(arg network_interface)"/>

File: legged_robot_description/g1_description/urdf/g1_29dof_lock_waist_rev_1_0_macro.urdf.xacro (robot description, xacro)
@@ -1,4 +1,4 @@
 <robot xmlns:xacro="http://ros.org/wiki/xacro">
-  <xacro:macro name="g1_29dof_lock_waist_rev_1_0" params="prefix">
+  <xacro:macro name="g1" params="prefix">
   <material name="dark">
     <color rgba="0.2 0.2 0.2 1"/>
@@ -25,5 +25,5 @@
       <origin xyz="0 0 0" rpy="0 0 0"/>
       <geometry>
-        <mesh filename="package://g1_description/meshes/pelvis.STL"/>
+        <mesh filename="package://g1_description/urdf/meshes/pelvis.STL"/>
       </geometry>
       <material name="dark"/>
@@ -39,12 +39,12 @@
       <origin xyz="0 0 0" rpy="0 0 0"/>
       <geometry>
-        <mesh filename="package://g1_description/meshes/pelvis_contour_link.STL"/>
-      </geometry>
-      <material name="white"/>
-    </visual>
-    <collision>
-      <origin xyz="0 0 0" rpy="0 0 0"/>
-      <geometry>
-        <mesh filename="package://g1_description/meshes/pelvis_contour_link.STL"/>
+        <mesh filename="package://g1_description/urdf/meshes/pelvis_contour_link.STL"/>
+      </geometry>
+      <material name="white"/>
+    </visual>
+    <collision>
+      <origin xyz="0 0 0" rpy="0 0 0"/>
+      <geometry>
+        <mesh filename="package://g1_description/urdf/meshes/pelvis_contour_link.STL"/>
       </geometry>
     </collision>
@@ -64,5 +64,5 @@
       <origin xyz="0 0 0" rpy="0 0 0"/>
       <geometry>
-        <mesh filename="package://g1_description/meshes/left_hip_pitch_link.STL"/>
+        <mesh filename="package://g1_description/urdf/meshes/left_hip_pitch_link.STL"/>
       </geometry>
       <material name="dark"/>
@@ -71,5 +71,5 @@
       <origin xyz="0 0 0" rpy="0 0 0"/>
       <geometry>
-        <mesh filename="package://g1_description/meshes/left_hip_pitch_link.STL"/>
+        <mesh filename="package://g1_description/urdf/meshes/left_hip_pitch_link.STL"/>
       </geometry>
     </collision>
@@ -91,12 +91,12 @@
       <origin xyz="0 0 0" rpy="0 0 0"/>
       <geometry>
-        <mesh filename="package://g1_description/meshes/left_hip_roll_link.STL"/>
-      </geometry>
-      <material name="white"/>
-    </visual>
-    <collision>
-      <origin xyz="0 0 0" rpy="0 0 0"/>
-      <geometry>
-        <mesh filename="package://g1_description/meshes/left_hip_roll_link.STL"/>
+        <mesh filename="package://g1_description/urdf/meshes/left_hip_roll_link.STL"/>
+      </geometry>
+      <material name="white"/>
+    </visual>
+    <collision>
+      <origin xyz="0 0 0" rpy="0 0 0"/>
+      <geometry>
+        <mesh filename="package://g1_description/urdf/meshes/left_hip_roll_link.STL"/>
       </geometry>
     </collision>
@@ -118,12 +118,12 @@
       <origin xyz="0 0 0" rpy="0 0 0"/>
       <geometry>
-        <mesh filename="package://g1_description/meshes/left_hip_yaw_link.STL"/>
-      </geometry>
-      <material name="white"/>
-    </visual>
-    <collision>
-      <origin xyz="0 0 0" rpy="0 0 0"/>
-      <geometry>
-        <mesh filename="package://g1_description/meshes/left_hip_yaw_link.STL"/>
+        <mesh filename="package://g1_description/urdf/meshes/left_hip_yaw_link.STL"/>
+      </geometry>
+      <material name="white"/>
+    </visual>
+    <collision>
+      <origin xyz="0 0 0" rpy="0 0 0"/>
+      <geometry>
+        <mesh filename="package://g1_description/urdf/meshes/left_hip_yaw_link.STL"/>
       </geometry>
     </collision>
@@ -145,12 +145,12 @@
       <origin xyz="0 0 0" rpy="0 0 0"/>
       <geometry>
-        <mesh filename="package://g1_description/meshes/left_knee_link.STL"/>
-      </geometry>
-      <material name="white"/>
-    </visual>
-    <collision>
-      <origin xyz="0 0 0" rpy="0 0 0"/>
-      <geometry>
-        <mesh filename="package://g1_description/meshes/left_knee_link.STL"/>
+        <mesh filename="package://g1_description/urdf/meshes/left_knee_link.STL"/>
+      </geometry>
+      <material name="white"/>
+    </visual>
+    <collision>
+      <origin xyz="0 0 0" rpy="0 0 0"/>
+      <geometry>
+        <mesh filename="package://g1_description/urdf/meshes/left_knee_link.STL"/>
       </geometry>
     </collision>
@@ -172,12 +172,12 @@
       <origin xyz="0 0 0" rpy="0 0 0"/>
       <geometry>
-        <mesh filename="package://g1_description/meshes/left_ankle_pitch_link.STL"/>
-      </geometry>
-      <material name="white"/>
-    </visual>
-    <collision>
-      <origin xyz="0 0 0" rpy="0 0 0"/>
-      <geometry>
-        <mesh filename="package://g1_description/meshes/left_ankle_pitch_link.STL"/>
+        <mesh filename="package://g1_description/urdf/meshes/left_ankle_pitch_link.STL"/>
+      </geometry>
+      <material name="white"/>
+    </visual>
+    <collision>
+      <origin xyz="0 0 0" rpy="0 0 0"/>
+      <geometry>
+        <mesh filename="package://g1_description/urdf/meshes/left_ankle_pitch_link.STL"/>
       </geometry>
     </collision>
@@ -199,5 +199,5 @@
       <origin xyz="0 0 0" rpy="0 0 0"/>
       <geometry>
-        <mesh filename="package://g1_description/meshes/left_ankle_roll_link.STL"/>
+        <mesh filename="package://g1_description/urdf/meshes/left_ankle_roll_link.STL"/>
       </geometry>
       <material name="dark"/>
@@ -244,5 +244,5 @@
       <origin xyz="0 0 0" rpy="0 0 0"/>
       <geometry>
-        <mesh filename="package://g1_description/meshes/right_hip_pitch_link.STL"/>
+        <mesh filename="package://g1_description/urdf/meshes/right_hip_pitch_link.STL"/>
       </geometry>
       <material name="dark"/>
@@ -251,5 +251,5 @@
       <origin xyz="0 0 0" rpy="0 0 0"/>
       <geometry>
-        <mesh filename="package://g1_description/meshes/right_hip_pitch_link.STL"/>
+        <mesh filename="package://g1_description/urdf/meshes/right_hip_pitch_link.STL"/>
       </geometry>
     </collision>
@@ -271,12 +271,12 @@
       <origin xyz="0 0 0" rpy="0 0 0"/>
       <geometry>
-        <mesh filename="package://g1_description/meshes/right_hip_roll_link.STL"/>
-      </geometry>
-      <material name="white"/>
-    </visual>
-    <collision>
-      <origin xyz="0 0 0" rpy="0 0 0"/>
-      <geometry>
-        <mesh filename="package://g1_description/meshes/right_hip_roll_link.STL"/>
+        <mesh filename="package://g1_description/urdf/meshes/right_hip_roll_link.STL"/>
+      </geometry>
+      <material name="white"/>
+    </visual>
+    <collision>
+      <origin xyz="0 0 0" rpy="0 0 0"/>
+      <geometry>
+        <mesh filename="package://g1_description/urdf/meshes/right_hip_roll_link.STL"/>
       </geometry>
     </collision>
@@ -298,12 +298,12 @@
       <origin xyz="0 0 0" rpy="0 0 0"/>
       <geometry>
-        <mesh filename="package://g1_description/meshes/right_hip_yaw_link.STL"/>
-      </geometry>
-      <material name="white"/>
-    </visual>
-    <collision>
-      <origin xyz="0 0 0" rpy="0 0 0"/>
-      <geometry>
-        <mesh filename="package://g1_description/meshes/right_hip_yaw_link.STL"/>
+        <mesh filename="package://g1_description/urdf/meshes/right_hip_yaw_link.STL"/>
+      </geometry>
+      <material name="white"/>
+    </visual>
+    <collision>
+      <origin xyz="0 0 0" rpy="0 0 0"/>
+      <geometry>
+        <mesh filename="package://g1_description/urdf/meshes/right_hip_yaw_link.STL"/>
       </geometry>
     </collision>
@@ -325,12 +325,12 @@
       <origin xyz="0 0 0" rpy="0 0 0"/>
       <geometry>
-        <mesh filename="package://g1_description/meshes/right_knee_link.STL"/>
-      </geometry>
-      <material name="white"/>
-    </visual>
-    <collision>
-      <origin xyz="0 0 0" rpy="0 0 0"/>
-      <geometry>
-        <mesh filename="package://g1_description/meshes/right_knee_link.STL"/>
+        <mesh filename="package://g1_description/urdf/meshes/right_knee_link.STL"/>
+      </geometry>
+      <material name="white"/>
+    </visual>
+    <collision>
+      <origin xyz="0 0 0" rpy="0 0 0"/>
+      <geometry>
+        <mesh filename="package://g1_description/urdf/meshes/right_knee_link.STL"/>
       </geometry>
     </collision>
@@ -352,12 +352,12 @@
       <origin xyz="0 0 0" rpy="0 0 0"/>
       <geometry>
-        <mesh filename="package://g1_description/meshes/right_ankle_pitch_link.STL"/>
-      </geometry>
-      <material name="white"/>
-    </visual>
-    <collision>
-      <origin xyz="0 0 0" rpy="0 0 0"/>
-      <geometry>
-        <mesh filename="package://g1_description/meshes/right_ankle_pitch_link.STL"/>
+        <mesh filename="package://g1_description/urdf/meshes/right_ankle_pitch_link.STL"/>
+      </geometry>
+      <material name="white"/>
+    </visual>
+    <collision>
+      <origin xyz="0 0 0" rpy="0 0 0"/>
+      <geometry>
+        <mesh filename="package://g1_description/urdf/meshes/right_ankle_pitch_link.STL"/>
       </geometry>
     </collision>
@@ -379,5 +379,5 @@
       <origin xyz="0 0 0" rpy="0 0 0"/>
       <geometry>
-        <mesh filename="package://g1_description/meshes/right_ankle_roll_link.STL"/>
+        <mesh filename="package://g1_description/urdf/meshes/right_ankle_roll_link.STL"/>
       </geometry>
       <material name="dark"/>
@@ -425,5 +425,5 @@
       <origin xyz="0 0 0" rpy="0 0 0"/>
       <geometry>
-        <mesh filename="package://g1_description/meshes/waist_yaw_link_rev_1_0.STL"/>
+        <mesh filename="package://g1_description/urdf/meshes/waist_yaw_link_rev_1_0.STL"/>
       </geometry>
       <material name="white"/>
@@ -446,5 +446,5 @@
       <origin xyz="0 0 0" rpy="0 0 0"/>
       <geometry>
-        <mesh filename="package://g1_description/meshes/waist_roll_link_rev_1_0.STL"/>
+        <mesh filename="package://g1_description/urdf/meshes/waist_roll_link_rev_1_0.STL"/>
       </geometry>
       <material name="white"/>
@@ -467,12 +467,12 @@
       <origin xyz="0 0 0" rpy="0 0 0"/>
       <geometry>
-        <mesh filename="package://g1_description/meshes/torso_link_rev_1_0.STL"/>
-      </geometry>
-      <material name="white"/>
-    </visual>
-    <collision>
-      <origin xyz="0 0 0" rpy="0 0 0"/>
-      <geometry>
-        <mesh filename="package://g1_description/meshes/torso_link_rev_1_0.STL"/>
+        <mesh filename="package://g1_description/urdf/meshes/torso_link_rev_1_0.STL"/>
+      </geometry>
+      <material name="white"/>
+    </visual>
+    <collision>
+      <origin xyz="0 0 0" rpy="0 0 0"/>
+      <geometry>
+        <mesh filename="package://g1_description/urdf/meshes/torso_link_rev_1_0.STL"/>
       </geometry>
     </collision>
@@ -500,5 +500,5 @@
       <origin xyz="0 0 0" rpy="0 0 0"/>
       <geometry>
-        <mesh filename="package://g1_description/meshes/logo_link.STL"/>
+        <mesh filename="package://g1_description/urdf/meshes/logo_link.STL"/>
       </geometry>
       <material name="dark"/>
@@ -507,5 +507,5 @@
       <origin xyz="0 0 0" rpy="0 0 0"/>
       <geometry>
-        <mesh filename="package://g1_description/meshes/logo_link.STL"/>
+        <mesh filename="package://g1_description/urdf/meshes/logo_link.STL"/>
       </geometry>
     </collision>
@@ -521,5 +521,5 @@
       <origin xyz="0 0 0" rpy="0 0 0"/>
       <geometry>
-        <mesh filename="package://g1_description/meshes/head_link.STL"/>
+        <mesh filename="package://g1_description/urdf/meshes/head_link.STL"/>
       </geometry>
       <material name="dark"/>
@@ -528,5 +528,5 @@
       <origin xyz="0 0 0" rpy="0 0 0"/>
       <geometry>
-        <mesh filename="package://g1_description/meshes/head_link.STL"/>
+        <mesh filename="package://g1_description/urdf/meshes/head_link.STL"/>
       </geometry>
     </collision>
@@ -574,5 +574,5 @@
       <origin xyz="0 0 0" rpy="0 0 0"/>
       <geometry>
-        <mesh filename="package://g1_description/meshes/left_shoulder_pitch_link.STL"/>
+        <mesh filename="package://g1_description/urdf/meshes/left_shoulder_pitch_link.STL"/>
       </geometry>
       <material name="white"/>
@@ -601,5 +601,5 @@
       <origin xyz="0 0 0" rpy="0 0 0"/>
       <geometry>
-        <mesh filename="package://g1_description/meshes/left_shoulder_roll_link.STL"/>
+        <mesh filename="package://g1_description/urdf/meshes/left_shoulder_roll_link.STL"/>
       </geometry>
       <material name="white"/>
@@ -628,12 +628,12 @@
       <origin xyz="0 0 0" rpy="0 0 0"/>
       <geometry>
-        <mesh filename="package://g1_description/meshes/left_shoulder_yaw_link.STL"/>
-      </geometry>
-      <material name="white"/>
-    </visual>
-    <collision>
-      <origin xyz="0 0 0" rpy="0 0 0"/>
-      <geometry>
-        <mesh filename="package://g1_description/meshes/left_shoulder_yaw_link.STL"/>
+        <mesh filename="package://g1_description/urdf/meshes/left_shoulder_yaw_link.STL"/>
+      </geometry>
+      <material name="white"/>
+    </visual>
+    <collision>
+      <origin xyz="0 0 0" rpy="0 0 0"/>
+      <geometry>
+        <mesh filename="package://g1_description/urdf/meshes/left_shoulder_yaw_link.STL"/>
       </geometry>
     </collision>
@@ -655,12 +655,12 @@
       <origin xyz="0 0 0" rpy="0 0 0"/>
       <geometry>
-        <mesh filename="package://g1_description/meshes/left_elbow_link.STL"/>
-      </geometry>
-      <material name="white"/>
-    </visual>
-    <collision>
-      <origin xyz="0 0 0" rpy="0 0 0"/>
-      <geometry>
-        <mesh filename="package://g1_description/meshes/left_elbow_link.STL"/>
+        <mesh filename="package://g1_description/urdf/meshes/left_elbow_link.STL"/>
+      </geometry>
+      <material name="white"/>
+    </visual>
+    <collision>
+      <origin xyz="0 0 0" rpy="0 0 0"/>
+      <geometry>
+        <mesh filename="package://g1_description/urdf/meshes/left_elbow_link.STL"/>
       </geometry>
     </collision>
@@ -689,12 +689,12 @@
       <origin xyz="0 0 0" rpy="0 0 0"/>
       <geometry>
-        <mesh filename="package://g1_description/meshes/left_wrist_roll_link.STL"/>
-      </geometry>
-      <material name="white"/>
-    </visual>
-    <collision>
-      <origin xyz="0 0 0" rpy="0 0 0"/>
-      <geometry>
-        <mesh filename="package://g1_description/meshes/left_wrist_roll_link.STL"/>
+        <mesh filename="package://g1_description/urdf/meshes/left_wrist_roll_link.STL"/>
+      </geometry>
+      <material name="white"/>
+    </visual>
+    <collision>
+      <origin xyz="0 0 0" rpy="0 0 0"/>
+      <geometry>
+        <mesh filename="package://g1_description/urdf/meshes/left_wrist_roll_link.STL"/>
       </geometry>
     </collision>
@@ -716,12 +716,12 @@
       <origin xyz="0 0 0" rpy="0 0 0"/>
       <geometry>
-        <mesh filename="package://g1_description/meshes/left_wrist_pitch_link.STL"/>
-      </geometry>
-      <material name="white"/>
-    </visual>
-    <collision>
-      <origin xyz="0 0 0" rpy="0 0 0"/>
-      <geometry>
-        <mesh filename="package://g1_description/meshes/left_wrist_pitch_link.STL"/>
+        <mesh filename="package://g1_description/urdf/meshes/left_wrist_pitch_link.STL"/>
+      </geometry>
+      <material name="white"/>
+    </visual>
+    <collision>
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