Commit message: new branch isaacsim-controller

File: legged_robot_description/g1_description/urdf/g1_29dof_lock_waist_rev_1_0.ros2_control.xacro (robot description, xacro)
@@ -1,535 +1,70 @@
 <?xml version="1.0"?>
 <robot xmlns:xacro="http://www.ros.org/wiki/xacro">
-  <xacro:macro name="g1_ros2_control" params="prefix network_interface:=lo">
-    <ros2_control name="g1_ros2_control" type="system" is_async="true">
+  <xacro:macro name="g1_ros2_control" params="prefix network_interface:=lo use_sim:=true">
+    <ros2_control name="g1_ros2_control" type="system">
       <hardware>
-        <plugin>legged_ros2_control/G1SystemInterface</plugin>
-        <param name="network_interface">${network_interface}</param>
+        <xacro:if value="${use_sim}">
+          <!-- Mode Isaac Sim -->
+          <plugin>topic_based_ros2_control/TopicBasedSystem</plugin>
+          <param name="joint_commands_topic">/joint_commands</param>
+          <param name="joint_states_topic">/joint_states</param>
+          <param name="imu_sensor_topic">/imu</param>
+        </xacro:if>
+        <xacro:unless value="${use_sim}">
+          <!-- Mode Mujoco and Real Robot -->
+          <plugin>legged_ros2_control/G1SystemInterface</plugin>
+          <param name="network_interface">${network_interface}</param>
+        </xacro:unless>
       </hardware>
-      <joint name="${prefix}left_hip_pitch_joint">
-        <command_interface name="position">
-          <param name="min">-2.5307</param>
-          <param name="max">2.8798</param>
-        </command_interface>
-        <command_interface name="velocity">
-          <param name="min">-32.0</param>
-          <param name="max">32.0</param>
-        </command_interface>
-        <command_interface name="effort">
-          <param name="min">-88.0</param>
-          <param name="max">88.0</param>
-        </command_interface>
-        <state_interface name="position">
-          <param name="initial_value">0.0</param>
-        </state_interface>
-        <state_interface name="velocity" />
-        <state_interface name="effort" />
-      </joint>
-      <joint name="${prefix}left_hip_roll_joint">
-        <command_interface name="position">
-          <param name="min">-0.5236</param>
-          <param name="max">2.9671</param>
-        </command_interface>
-        <command_interface name="velocity">
-          <param name="min">-20.0</param>
-          <param name="max">20.0</param>
-        </command_interface>
-        <command_interface name="effort">
-          <param name="min">-139.0</param>
-          <param name="max">139.0</param>
-        </command_interface>
-        <state_interface name="position">
-          <param name="initial_value">0.0</param>
-        </state_interface>
-        <state_interface name="velocity" />
-        <state_interface name="effort" />
-      </joint>
-      <joint name="${prefix}left_hip_yaw_joint">
-        <command_interface name="position">
-          <param name="min">-2.7576</param>
-          <param name="max">2.7576</param>
-        </command_interface>
-        <command_interface name="velocity">
-          <param name="min">-32.0</param>
-          <param name="max">32.0</param>
-        </command_interface>
-        <command_interface name="effort">
-          <param name="min">-88.0</param>
-          <param name="max">88.0</param>
-        </command_interface>
-        <state_interface name="position">
-          <param name="initial_value">0.0</param>
-        </state_interface>
-        <state_interface name="velocity" />
-        <state_interface name="effort" />
-      </joint>
-      <joint name="${prefix}left_knee_joint">
-        <command_interface name="position">
-          <param name="min">-0.087267</param>
-          <param name="max">2.8798</param>
-        </command_interface>
-        <command_interface name="velocity">
-          <param name="min">-20.0</param>
-          <param name="max">20.0</param>
-        </command_interface>
-        <command_interface name="effort">
-          <param name="min">-139.0</param>
-          <param name="max">139.0</param>
-        </command_interface>
-        <state_interface name="position">
-          <param name="initial_value">0.0</param>
-        </state_interface>
-        <state_interface name="velocity" />
-        <state_interface name="effort" />
-      </joint>
-      <joint name="${prefix}left_ankle_pitch_joint">
-        <command_interface name="position">
-          <param name="min">-0.87267</param>
-          <param name="max">0.5236</param>
-        </command_interface>
-        <command_interface name="velocity">
-          <param name="min">-30.0</param>
-          <param name="max">30.0</param>
-        </command_interface>
-        <command_interface name="effort">
-          <param name="min">-35.0</param>
-          <param name="max">35.0</param>
-        </command_interface>
-        <state_interface name="position">
-          <param name="initial_value">0.0</param>
-        </state_interface>
-        <state_interface name="velocity" />
-        <state_interface name="effort" />
-      </joint>
-      <joint name="${prefix}left_ankle_roll_joint">
-        <command_interface name="position">
-          <param name="min">-0.2618</param>
-          <param name="max">0.2618</param>
-        </command_interface>
-        <command_interface name="velocity">
-          <param name="min">-30.0</param>
-          <param name="max">30.0</param>
-        </command_interface>
-        <command_interface name="effort">
-          <param name="min">-35.0</param>
-          <param name="max">35.0</param>
-        </command_interface>
-        <state_interface name="position">
-          <param name="initial_value">0.0</param>
-        </state_interface>
-        <state_interface name="velocity" />
-        <state_interface name="effort" />
-      </joint>
-      <joint name="${prefix}right_hip_pitch_joint">
-        <command_interface name="position">
-          <param name="min">-2.5307</param>
-          <param name="max">2.8798</param>
-        </command_interface>
-        <command_interface name="velocity">
-          <param name="min">-32.0</param>
-          <param name="max">32.0</param>
-        </command_interface>
-        <command_interface name="effort">
-          <param name="min">-88.0</param>
-          <param name="max">88.0</param>
-        </command_interface>
-        <state_interface name="position">
-          <param name="initial_value">0.0</param>
-        </state_interface>
-        <state_interface name="velocity" />
-        <state_interface name="effort" />
-      </joint>
-      <joint name="${prefix}right_hip_roll_joint">
-        <command_interface name="position">
-          <param name="min">-2.9671</param>
-          <param name="max">0.5236</param>
-        </command_interface>
-        <command_interface name="velocity">
-          <param name="min">-20.0</param>
-          <param name="max">20.0</param>
-        </command_interface>
-        <command_interface name="effort">
-          <param name="min">-139.0</param>
-          <param name="max">139.0</param>
-        </command_interface>
-        <state_interface name="position">
-          <param name="initial_value">0.0</param>
-        </state_interface>
-        <state_interface name="velocity" />
-        <state_interface name="effort" />
-      </joint>
-      <joint name="${prefix}right_hip_yaw_joint">
-        <command_interface name="position">
-          <param name="min">-2.7576</param>
-          <param name="max">2.7576</param>
-        </command_interface>
-        <command_interface name="velocity">
-          <param name="min">-32.0</param>
-          <param name="max">32.0</param>
-        </command_interface>
-        <command_interface name="effort">
-          <param name="min">-88.0</param>
-          <param name="max">88.0</param>
-        </command_interface>
-        <state_interface name="position">
-          <param name="initial_value">0.0</param>
-        </state_interface>
-        <state_interface name="velocity" />
-        <state_interface name="effort" />
-      </joint>
-      <joint name="${prefix}right_knee_joint">
-        <command_interface name="position">
-          <param name="min">-0.087267</param>
-          <param name="max">2.8798</param>
-        </command_interface>
-        <command_interface name="velocity">
-          <param name="min">-20.0</param>
-          <param name="max">20.0</param>
-        </command_interface>
-        <command_interface name="effort">
-          <param name="min">-139.0</param>
-          <param name="max">139.0</param>
-        </command_interface>
-        <state_interface name="position">
-          <param name="initial_value">0.0</param>
-        </state_interface>
-        <state_interface name="velocity" />
-        <state_interface name="effort" />
-      </joint>
-      <joint name="${prefix}right_ankle_pitch_joint">
-        <command_interface name="position">
-          <param name="min">-0.87267</param>
-          <param name="max">0.5236</param>
-        </command_interface>
-        <command_interface name="velocity">
-          <param name="min">-30.0</param>
-          <param name="max">30.0</param>
-        </command_interface>
-        <command_interface name="effort">
-          <param name="min">-35.0</param>
-          <param name="max">35.0</param>
-        </command_interface>
-        <state_interface name="position">
-          <param name="initial_value">0.0</param>
-        </state_interface>
-        <state_interface name="velocity" />
-        <state_interface name="effort" />
-      </joint>
-      <joint name="${prefix}right_ankle_roll_joint">
-        <command_interface name="position">
-          <param name="min">-0.2618</param>
-          <param name="max">0.2618</param>
-        </command_interface>
-        <command_interface name="velocity">
-          <param name="min">-30.0</param>
-          <param name="max">30.0</param>
-        </command_interface>
-        <command_interface name="effort">
-          <param name="min">-35.0</param>
-          <param name="max">35.0</param>
-        </command_interface>
-        <state_interface name="position">
-          <param name="initial_value">0.0</param>
-        </state_interface>
-        <state_interface name="velocity" />
-        <state_interface name="effort" />
-      </joint>
-      <joint name="${prefix}waist_yaw_joint">
-        <command_interface name="position">
-          <param name="min">-2.618</param>
-          <param name="max">2.618</param>
-        </command_interface>
-        <command_interface name="velocity">
-          <param name="min">-32.0</param>
-          <param name="max">32.0</param>
-        </command_interface>
-        <command_interface name="effort">
-          <param name="min">-88.0</param>
-          <param name="max">88.0</param>
-        </command_interface>
-        <state_interface name="position">
-          <param name="initial_value">0.0</param>
-        </state_interface>
-        <state_interface name="velocity" />
-        <state_interface name="effort" />
-      </joint>
-      <joint name="${prefix}left_shoulder_pitch_joint">
-        <command_interface name="position">
-          <param name="min">-3.0892</param>
-          <param name="max">2.6704</param>
-        </command_interface>
-        <command_interface name="velocity">
-          <param name="min">-37.0</param>
-          <param name="max">37.0</param>
-        </command_interface>
-        <command_interface name="effort">
-          <param name="min">-25.0</param>
-          <param name="max">25.0</param>
-        </command_interface>
-        <state_interface name="position">
-          <param name="initial_value">0.0</param>
-        </state_interface>
-        <state_interface name="velocity" />
-        <state_interface name="effort" />
-      </joint>
-      <joint name="${prefix}left_shoulder_roll_joint">
-        <command_interface name="position">
-          <param name="min">-1.5882</param>
-          <param name="max">2.2515</param>
-        </command_interface>
-        <command_interface name="velocity">
-          <param name="min">-37.0</param>
-          <param name="max">37.0</param>
-        </command_interface>
-        <command_interface name="effort">
-          <param name="min">-25.0</param>
-          <param name="max">25.0</param>
-        </command_interface>
-        <state_interface name="position">
-          <param name="initial_value">0.0</param>
-        </state_interface>
-        <state_interface name="velocity" />
-        <state_interface name="effort" />
-      </joint>
-      <joint name="${prefix}left_shoulder_yaw_joint">
-        <command_interface name="position">
-          <param name="min">-2.618</param>
-          <param name="max">2.618</param>
-        </command_interface>
-        <command_interface name="velocity">
-          <param name="min">-37.0</param>
-          <param name="max">37.0</param>
-        </command_interface>
-        <command_interface name="effort">
-          <param name="min">-25.0</param>
-          <param name="max">25.0</param>
-        </command_interface>
-        <state_interface name="position">
-          <param name="initial_value">0.0</param>
-        </state_interface>
-        <state_interface name="velocity" />
-        <state_interface name="effort" />
-      </joint>
-      <joint name="${prefix}left_elbow_joint">
-        <command_interface name="position">
-          <param name="min">-1.0472</param>
-          <param name="max">2.0944</param>
-        </command_interface>
-        <command_interface name="velocity">
-          <param name="min">-37.0</param>
-          <param name="max">37.0</param>
-        </command_interface>
-        <command_interface name="effort">
-          <param name="min">-25.0</param>
-          <param name="max">25.0</param>
-        </command_interface>
-        <state_interface name="position">
-          <param name="initial_value">0.0</param>
-        </state_interface>
-        <state_interface name="velocity" />
-        <state_interface name="effort" />
-      </joint>
-      <joint name="${prefix}left_wrist_roll_joint">
-        <command_interface name="position">
-          <param name="min">-1.972222054</param>
-          <param name="max">1.972222054</param>
-        </command_interface>
-        <command_interface name="velocity">
-          <param name="min">-37.0</param>
-          <param name="max">37.0</param>
-        </command_interface>
-        <command_interface name="effort">
-          <param name="min">-25.0</param>
-          <param name="max">25.0</param>
-        </command_interface>
-        <state_interface name="position">
-          <param name="initial_value">0.0</param>
-        </state_interface>
-        <state_interface name="velocity" />
-        <state_interface name="effort" />
-      </joint>
-      <joint name="${prefix}left_wrist_pitch_joint">
-        <command_interface name="position">
-          <param name="min">-1.614429558</param>
-          <param name="max">1.614429558</param>
-        </command_interface>
-        <command_interface name="velocity">
-          <param name="min">-22.0</param>
-          <param name="max">22.0</param>
-        </command_interface>
-        <command_interface name="effort">
-          <param name="min">-5.0</param>
-          <param name="max">5.0</param>
-        </command_interface>
-        <state_interface name="position">
-          <param name="initial_value">0.0</param>
-        </state_interface>
-        <state_interface name="velocity" />
-        <state_interface name="effort" />
-      </joint>
-      <joint name="${prefix}left_wrist_yaw_joint">
-        <command_interface name="position">
-          <param name="min">-1.614429558</param>
-          <param name="max">1.614429558</param>
-        </command_interface>
-        <command_interface name="velocity">
-          <param name="min">-22.0</param>
-          <param name="max">22.0</param>
-        </command_interface>
-        <command_interface name="effort">
-          <param name="min">-5.0</param>
-          <param name="max">5.0</param>
-        </command_interface>
-        <state_interface name="position">
-          <param name="initial_value">0.0</param>
-        </state_interface>
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
File: legged_robot_description/g1_description/urdf/g1_29dof_lock_waist_rev_1_0.urdf.xacro (robot description, xacro)
@@ -3,4 +3,5 @@
   <xacro:arg name="prefix" default="" />
   <xacro:arg name="network_interface" default="lo" />
+  <xacro:arg name="use_sim" default="true" />
   <xacro:include filename="$(find g1_description)/urdf/g1_29dof_lock_waist_rev_1_0_macro.urdf.xacro" />
   <xacro:include filename="$(find g1_description)/urdf/g1_29dof_lock_waist_rev_1_0.ros2_control.xacro" />
@@ -8,4 +9,5 @@
   <xacro:g1_ros2_control
     prefix="$(arg prefix)"
-    network_interface="$(arg network_interface)"/>
+    network_interface="$(arg network_interface)"
+    use_sim="$(arg use_sim)"/>
 </robot>

File: legged_robot_description/g1_description/urdf/g1_29dof_lock_waist_rev_1_0_macro.urdf.xacro (robot description, xacro)
@@ -451,5 +451,5 @@
     </visual>
   </link>
-  <joint name="${prefix}waist_roll_joint" type="fixed">
+  <joint name="${prefix}waist_roll_joint" type="revolute">
     <origin xyz="-0.0039635 0 0.044" rpy="0 0 0"/>
     <parent link="${prefix}waist_yaw_link"/>
@@ -478,5 +478,5 @@
     </collision>
   </link>
-  <joint name="${prefix}waist_pitch_joint" type="fixed">
+  <joint name="${prefix}waist_pitch_joint" type="revolute">
     <origin xyz="0 0 0" rpy="0 0 0"/>
     <parent link="${prefix}waist_roll_link"/>

Commit message: update dds domain id

File: legged_robot_description/g1_description/urdf/g1_29dof_lock_waist_rev_1_0.ros2_control.xacro (robot description, xacro)
@@ -1,9 +1,9 @@
 <?xml version="1.0"?>
 <robot xmlns:xacro="http://www.ros.org/wiki/xacro">
-  <xacro:macro name="g1_ros2_control" params="prefix network_interface:=lo use_sim:=true">
+  <xacro:macro name="g1_ros2_control" params="prefix network_interface:=lo use_sim:=true domain_id:=0">
     <ros2_control name="g1_ros2_control" type="system">
       <hardware>
         <xacro:if value="${use_sim}">
-          <!-- Mode Isaac Sim -->
+          <!-- Isaac-style sim: topics /joint_commands, /joint_states (not MuJoCo DDS). -->
           <plugin>topic_based_ros2_control/TopicBasedSystem</plugin>
           <param name="joint_commands_topic">/joint_commands</param>
@@ -12,7 +12,8 @@
         </xacro:if>
         <xacro:unless value="${use_sim}">
-          <!-- Mode Mujoco and Real Robot -->
+          <!-- MuJoCo (unitree_mujoco DDS) and real robot -->
           <plugin>legged_ros2_control/G1SystemInterface</plugin>
           <param name="network_interface">${network_interface}</param>
+          <param name="domain_id">${domain_id}</param>
         </xacro:unless>
       </hardware>

File: legged_robot_description/g1_description/urdf/g1_29dof_lock_waist_rev_1_0.urdf.xacro (robot description, xacro)
@@ -3,4 +3,5 @@
   <xacro:arg name="prefix" default="" />
   <xacro:arg name="network_interface" default="lo" />
+  <xacro:arg name="domain_id" default="0" />
   <xacro:arg name="use_sim" default="true" />
   <xacro:arg name="use_mock_components" default="false" />
@@ -11,4 +12,5 @@
     prefix="$(arg prefix)"
     network_interface="$(arg network_interface)"
+    domain_id="$(arg domain_id)"
     use_sim="$(arg use_sim)"/>
    <!-- Gipper URDF -->
