Commit message: update control isaacsim gripper

File: legged_robot_description/g1_description/urdf/inspire_gripper/inspire_gripper.ros2_control.xacro (robot description, xacro)
@@ -4,5 +4,5 @@
         name
         prefix
-        use_sim:=false
+        use_sim:=true
         use_mock_components:=false
         serial_port:=/dev/ttyUSB0
@@ -11,7 +11,15 @@
         <ros2_control name="${name}_gripper_hardware" type="system">
             <hardware>
-                <xacro:if value="${use_sim or use_mock_components}">
+                <!-- 1. Mode Isaac Sim: Using TopicBasedSystem -->
+                <xacro:if value="${use_sim}">
+                    <plugin>topic_based_ros2_control/TopicBasedSystem</plugin>
+                    <param name="joint_commands_topic">/${prefix}gripper_commands</param>
+                    <param name="joint_states_topic">/${prefix}gripper_states</param>
+                </xacro:if>
+                <!-- 2. Mode Mock -->
+                <xacro:if value="${use_mock_components and not use_sim}">
                     <plugin>mock_components/GenericSystem</plugin>
                 </xacro:if>
+                <!-- 3. Mode Real Hardware -->
                 <xacro:unless value="${use_sim or use_mock_components}">
                     <plugin>vm_ros2_control/InspireGripperHardwareInterface</plugin>
@@ -20,5 +28,6 @@
                 </xacro:unless>
             </hardware>
-            <joint name="${prefix}inspire_gripper_joint1">
+            <!-- Main joint (Joint 1) -->
+            <joint name="inspire_gripper_joint1">
                 <command_interface name="position" />
                 <state_interface name="position">
@@ -29,8 +38,9 @@
                 </state_interface>
             </joint>
+            <!-- Mimic Joint-->
             <xacro:if value="${use_sim or use_mock_components}">
                 <xacro:macro name="mimic_joint_hw" params="joint_num mult">
-                    <joint name="${prefix}inspire_gripper_joint${joint_num}">
-                        <param name="mimic">${prefix}inspire_gripper_joint1</param>
+                    <joint name="inspire_gripper_joint${joint_num}">
+                        <param name="mimic">inspire_gripper_joint1</param>
                         <param name="multiplier">${mult}</param>
                         <command_interface name="position" />
@@ -45,4 +55,5 @@
                 <xacro:mimic_joint_hw joint_num="6" mult="1"/>
             </xacro:if>
+            <!-- GPIO only valid on real robot -->
             <xacro:unless value="${use_sim or use_mock_components}">
                 <gpio name="${prefix}reactivate_gripper">

File: legged_robot_description/g1_description/urdf/inspire_gripper/inspire_gripper_description.xacro (robot description, xacro)
@@ -3,5 +3,5 @@
   <xacro:macro name="inspire_gripper_description" params="prefix">
     <!-- BASE LINK -->
-    <link name="${prefix}inspire_gripper_baselink">
+    <link name="$inspire_gripper_baselink">
       <inertial>
         <origin xyz="1.5645E-05 -4.1838E-06 0.038" rpy="0 0 0" />
@@ -24,5 +24,5 @@
     </link>
     <!-- LINK 1 -->
-    <link name="${prefix}inspire_gripper_link1">
+    <link name="$inspire_gripper_link1">
       <inertial>
         <origin xyz="0.0087669 0.009 0.013992" rpy="0 0 0" />
@@ -44,8 +44,8 @@
     </link>
     <!-- JOINT 1 (Main joint) -->
-    <joint name="${prefix}inspire_gripper_joint1" type="revolute">
+    <joint name="$inspire_gripper_joint1" type="revolute">
       <origin xyz="-0.04 -0.009 0.079" rpy="0 0 0" />
-      <parent link="${prefix}inspire_gripper_baselink" />
-      <child link="${prefix}inspire_gripper_link1" />
+      <parent link="$inspire_gripper_baselink" />
+      <child link="$inspire_gripper_link1" />
       <axis xyz="0 -1 0" />
       <limit lower="0" upper="0.82" effort="1" velocity="0.5" />
@@ -53,5 +53,5 @@
     </joint>
     <!-- LINK 5 -->
-    <link name="${prefix}inspire_gripper_link5">
+    <link name="$inspire_gripper_link5">
       <inertial>
         <origin xyz="0.011864 0.006 0.011367" rpy="0 0 0" />
@@ -73,15 +73,15 @@
     </link>
     <!-- JOINT 5 (Mimic) -->
-    <joint name="${prefix}inspire_gripper_joint5" type="revolute">
+    <joint name="$inspire_gripper_joint5" type="revolute">
       <origin xyz="0.0223 0.003 0.035591" rpy="0 0 0" />
-      <parent link="${prefix}inspire_gripper_link1" />
-      <child link="${prefix}inspire_gripper_link5" />
+      <parent link="$inspire_gripper_link1" />
+      <child link="$inspire_gripper_link5" />
       <axis xyz="0 1 0" />
       <limit lower="0" upper="0.82" effort="1" velocity="0.5" />
       <dynamics damping="0.1" friction="0.1"/>
-      <mimic joint="${prefix}inspire_gripper_joint1"/>
+      <mimic joint="$inspire_gripper_joint1"/>
     </joint>
     <!-- LINK 2 -->
-    <link name="${prefix}inspire_gripper_link2">
+    <link name="$inspire_gripper_link2">
       <inertial>
         <origin xyz="0.0087435 0.009 0.013955" rpy="0 0 0" />
@@ -103,15 +103,15 @@
     </link>
     <!-- JOINT 2 (Mimic) -->
-    <joint name="${prefix}inspire_gripper_joint2" type="revolute">
+    <joint name="$inspire_gripper_joint2" type="revolute">
       <origin xyz="-0.03 -0.009 0.081" rpy="0 0 0" />
-      <parent link="${prefix}inspire_gripper_baselink" />
-      <child link="${prefix}inspire_gripper_link2" />
-      <axis xyz="0 -1 0" />
-      <limit lower="0" upper="0.82" effort="1" velocity="0.5" />
-      <dynamics damping="0.1" friction="0.1"/>
-      <mimic joint="${prefix}inspire_gripper_joint1"/>
+      <parent link="$inspire_gripper_baselink" />
+      <child link="$inspire_gripper_link2" />
+      <axis xyz="0 -1 0" />
+      <limit lower="0" upper="0.82" effort="1" velocity="0.5" />
+      <dynamics damping="0.1" friction="0.1"/>
+      <mimic joint="$inspire_gripper_joint1"/>
     </joint>
     <!-- LINK 3 -->
-    <link name="${prefix}inspire_gripper_link3">
+    <link name="$inspire_gripper_link3">
       <inertial>
         <origin xyz="-0.0087435 0.009 0.013955" rpy="0 0 0" />
@@ -133,15 +133,15 @@
     </link>
     <!-- JOINT 3 (Mimic) -->
-    <joint name="${prefix}inspire_gripper_joint3" type="revolute">
+    <joint name="$inspire_gripper_joint3" type="revolute">
       <origin xyz="0.03 -0.009 0.081" rpy="0 0 0" />
-      <parent link="${prefix}inspire_gripper_baselink" />
-      <child link="${prefix}inspire_gripper_link3" />
+      <parent link="$inspire_gripper_baselink" />
+      <child link="$inspire_gripper_link3" />
       <axis xyz="0 -1 0" />
       <limit lower="-0.82" upper="0" effort="1" velocity="0.5" />
       <dynamics damping="0.1" friction="0.1"/>
-      <mimic joint="${prefix}inspire_gripper_joint1" multiplier="-1" offset="0"/>
+      <mimic joint="$inspire_gripper_joint1" multiplier="-1" offset="0"/>
     </joint>
     <!-- LINK 4 -->
-    <link name="${prefix}inspire_gripper_link4">
+    <link name="$inspire_gripper_link4">
       <inertial>
         <origin xyz="-0.0087669 0.009 0.013992" rpy="0 0 0" />
@@ -163,15 +163,15 @@
     </link>
     <!-- JOINT 4 (Mimic) -->
-    <joint name="${prefix}inspire_gripper_joint4" type="revolute">
+    <joint name="$inspire_gripper_joint4" type="revolute">
       <origin xyz="0.04 -0.009 0.079" rpy="0 0 0" />
-      <parent link="${prefix}inspire_gripper_baselink" />
-      <child link="${prefix}inspire_gripper_link4" />
+      <parent link="$inspire_gripper_baselink" />
+      <child link="$inspire_gripper_link4" />
       <axis xyz="0 -1 0" />
       <limit lower="-0.82" upper="0" effort="1" velocity="0.5" />
       <dynamics damping="0.1" friction="0.1"/>
-      <mimic joint="${prefix}inspire_gripper_joint1" multiplier="-1" offset="0"/>
+      <mimic joint="$inspire_gripper_joint1" multiplier="-1" offset="0"/>
     </joint>
     <!-- LINK 6 -->
-    <link name="${prefix}inspire_gripper_link6">
+    <link name="$inspire_gripper_link6">
       <inertial>
         <origin xyz="-0.011864 0.006 0.011367" rpy="0 0 0" />
@@ -193,20 +193,20 @@
     </link>
     <!-- JOINT 6 (Mimic) -->
-    <joint name="${prefix}inspire_gripper_joint6" type="revolute">
+    <joint name="$inspire_gripper_joint6" type="revolute">
       <origin xyz="-0.0223 0.003 0.035591" rpy="0 0 0" />
-      <parent link="${prefix}inspire_gripper_link4" />
-      <child link="${prefix}inspire_gripper_link6" />
-      <axis xyz="0 -1 0" />
-      <limit lower="0" upper="0.82" effort="1" velocity="0.5" />
-      <dynamics damping="0.1" friction="0.1"/>
-      <mimic joint="${prefix}inspire_gripper_joint1"/>
+      <parent link="$inspire_gripper_link4" />
+      <child link="$inspire_gripper_link6" />
+      <axis xyz="0 -1 0" />
+      <limit lower="0" upper="0.82" effort="1" velocity="0.5" />
+      <dynamics damping="0.1" friction="0.1"/>
+      <mimic joint="$inspire_gripper_joint1"/>
     </joint>
     <!-- TRANSMISSION -->
-    <transmission name="${prefix}gripper_finger1_trans">
+    <transmission name="$gripper_finger1_trans">
       <type>transmission_interface/SimpleTransmission</type>
-      <joint name="${prefix}inspire_gripper_joint1">
+      <joint name="$inspire_gripper_joint1">
         <hardwareInterface>PositionJointInterface</hardwareInterface>
       </joint>
-      <actuator name="${prefix}gripper_finger1_motor">
+      <actuator name="$gripper_finger1_motor">
         <mechanicalReduction>1</mechanicalReduction>
         <hardwareInterface>PositionJointInterface</hardwareInterface>

File: legged_robot_description/g1_description/urdf/inspire_gripper_macro.xacro (robot description, xacro)
@@ -4,13 +4,14 @@
   <xacro:include filename="$(find g1_description)/urdf/inspire_gripper/inspire_gripper.ros2_control.xacro" />
   <xacro:macro name="inspire_gripper" params="name parent_link use_sim use_mock_components:=false serial_port *origin">
-    <xacro:inspire_gripper_description prefix="${name}_" />
-    <joint name="${name}_gripper_fix_joint" type="fixed">
+    <xacro:property name="gripper_prefix" value="${name}_" />
+    <xacro:inspire_gripper_description prefix="${gripper_prefix}" />
+    <joint name="${gripper_prefix}gripper_fix_joint" type="fixed">
       <xacro:insert_block name="origin" />
       <parent link="${parent_link}" />
-      <child link="${name}_inspire_gripper_baselink" />
+      <child link="${gripper_prefix}inspire_gripper_baselink" />
     </joint>
     <xacro:inspire_gripper_ros2_control
         name="${name}"
-        prefix="${name}_"
+        prefix="${gripper_prefix}"
         use_sim="${use_sim}"
         use_mock_components="${use_mock_components}"
